File: MD_Controller.sch (KiCad schematic (older format))
At the start: 66 parts, among them U1 power_connector, U2 CAN__connector, U3 potentio__connector, U4 encoder_connector, U5 NJM7800SDL1, U6 NJM7800SDL1, U7 dipSW, U8 power_connector

Commit message: 2.0.0
ネットリストの生成まで終了
Parts:
- removed U1, U8: power_connector, Connectors_JST:JST_XH_S02B-XH-A_02x2.50mm_Angled, symbol power_connector
- added D11, D12: LED, LEDs:LED_D5.0mm_FlatTop, symbol LED
- added JP1, JP2, JP3: JUMPER, Pin_Headers:Pin_Header_Straight_1x02_Pitch2.54mm, symbol JUMPER
- added R30, R31: R, Resistors_SMD:R_0603_HandSoldering, symbol R
- added U1, U8: XH_2, Connectors_JST:JST_XH_S02B-XH-A_02x2.50mm_Angled, symbol XH_2
- added U10, U9: XH_4, Connectors_JST:JST_XH_S04B-XH-A_04x2.50mm_Angled, symbol XH_4
- added U11: XH_3, Connectors_JST:JST_XH_S03B-XH-A_03x2.50mm_Angled, symbol XH_3
- D10, D3, D4, D5, D6, D7, D8, D9: footprint LEDs:LED_1206 -> LEDs:LED_0603_HandSoldering
- R1, R10, R11, R12, R13, R14, R15, R16, R17, R18, R19, R2, R20, R21, R22, R23, R24, R25, R26, R27, R28, R29, R3, R4, R5, R6, R7, R8, R9: footprint Resistors_SMD:R_1206_HandSoldering -> Resistors_SMD:R_0603_HandSoldering
- renumbered minibed to minibed1
Connections:
- net labels added: CS_1, CS_2, p10, p11, p15, p17
- wire segments 219 -> 253
- no-connect marks 39 -> 33
Other:
- moved on the sheet: D2, R1, R2, U2, U7, minibed1

Commit message: 2.0.1
入力ポートの増設
電流センサの外部出力ポートの増設
UARTポートの増設
Parts:
- removed JP1, JP2, JP3: JUMPER, Pin_Headers:Pin_Header_Straight_1x02_Pitch2.54mm, symbol JUMPER
- added U12: XH_3, Connectors_JST:JST_XH_S03B-XH-A_03x2.50mm_Angled, symbol XH_3
- D1: footprint LEDs:LED_1206 -> LEDs:LED_0603_HandSoldering
Connections:
- net CS_1: now also U12.2
- net CS_2: now also U12.1
- net GND: now also U12.3
- net GNDA: now also R10.2, R11.2, R6.2, R7.2, R8.2, R9.2; no longer D10.1 (K), D5.1 (K), D6.1 (K), D7.1 (K), D8.1 (K), D9.1 (K)
- net p0: now also D5.2 (A); no longer R6.1
- net p24: now also D7.2 (A); no longer R8.1
- net p25: now also D6.2 (A); no longer R7.1
- net p7: now also D10.2 (A); no longer R11.1
- net p8: now also D9.2 (A); no longer R10.1
- net p9: now also D8.2 (A); no longer R9.1
- net p10: no longer names the net of minibed1.21 (p10)
- net p11: no longer names the net of minibed1.22 (p11)
- new net: D5.1 (K), R6.1
- new net: D6.1 (K), R7.1
- new net: D7.1 (K), R8.1
- new net: D8.1 (K), R9.1
- new net: D9.1 (K), R10.1
- new net: D10.1 (K), R11.1
- no-connect marks 33 -> 35
Other:
- moved on the sheet: D10, D5, D6, D7, D8, D9, R10, R11, R6, R7, R8, R9
